File: Hardware/led_circle.kicad_sch (KiCad schematic)
At the start: 59 parts

Commit message: Added ESP32-WROOM
Parts:
- D1, D10, D11, D12, D13, D14, D15, D16, D17, D18, D19, D2, D20, D21, D22, D23, D24, D25, D26, D27, D28, D29, D3, D30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: LCSC C114592 -> (none); lcsc_new C114592 -> (none)
