File: Hardware/Project.kicad_pcb (KiCad board)
At the start: 4 copper layers, 230 x 230 mm, 196 parts, among them IC1 ESP32-S3-WROOM-1-N8, J1 USB_C_2.0, SW1 B3U-1000P, SW2 B3U-1000P, U2 TLV1117LV33DCYR

Commit message: Finished layout
Parts:
- C1, C2, C3, C4, D175, D176, D180, F3, IC1, R1, R2, U2: moved to B.Cu
- moved SW1 108.3 mm to (247.4, 332.0), turned to 90 degrees
- moved R4 104.8 mm to (244.8, 333.5), turned to 90 degrees
- moved R3 104.5 mm to (244.9, 330.4), turned to 90 degrees
- moved R2 98.2 mm to (251.2, 326.1), turned to 180 degrees
- moved D180 97.1 mm to (245.0, 324.9), turned to 90 degrees
- moved C1 96.3 mm to (234.6, 290.9), turned to 180 degrees
- moved C2 95.5 mm to (234.6, 289.4), turned to 180 degrees
- moved SW2 93.1 mm to (262.7, 332.0), turned to 90 degrees
- moved D175 92.3 mm to (251.5, 324.6)
- moved C3 89.2 mm to (251.9, 321.8), turned to 90 degrees
- moved J1 89.0 mm to (255.1, 331.7)
- moved U2 88.0 mm to (246.7, 319.7), turned to 180 degrees
- moved C4 86.0 mm to (252.0, 317.6), turned to 90 degrees
- moved R6 85.2 mm to (265.3, 333.5), turned to 90 degrees
- moved R5 84.9 mm to (265.3, 330.5), turned to 90 degrees
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Connections:
- IC1 pad 10: unconnected-(IC1-IO17-Pad10) -> LED_SEGMENTS
- IC1 pad 11: unconnected-(IC1-IO18-Pad11) -> LED_CIRCLE
- IC1 pad 38: LED_SEGMENTS -> unconnected-(IC1-IO2-Pad38)
- IC1 pad 39: LED_CIRCLE -> unconnected-(IC1-IO1-Pad39)
Routing:
- net LED_CIRCLE: track 1.10 -> 267.6 mm
- net +5V: track 245.5 -> 5.57 mm, vias 0 -> 175
- net LED_SEGMENTS: track 6.49 -> 119.0 mm
- net +3V3: track 0.00 -> 86.7 mm, vias 0 -> 2
- net GND: track 86.7 -> 5.27 mm, vias 170 -> 189
- net USB_N: track 0.00 -> 51.0 mm, vias 0 -> 2
- net USB_P: track 0.00 -> 49.0 mm, vias 0 -> 2
- net ESP_EN: track 0.00 -> 47.7 mm, vias 0 -> 1
- net BOOT0: track 0.00 -> 38.4 mm, vias 0 -> 1
- net Net-(F3-Pad2): track 0.00 -> 12.9 mm, vias 0 -> 1
- net Net-(J1-CC1): track 0.00 -> 3.47 mm, vias 0 -> 1
- net Net-(J1-CC2): track 0.00 -> 2.93 mm, vias 0 -> 1
- net Net-(SW1-A): track 0.00 -> 2.85 mm
- net Net-(SW2-A): track 0.00 -> 2.84 mm
